File: NimbusV1_Flight_Computer.kicad_sch (KiCad schematic)
At the start: 27 parts, among them J1 Pyro1, J2 Pyro2, J3 Pyro3, J4 Pyro4, Q1 IRF540N, Q2 IRF540N, Q3 IRF540N, Q4 IRF540N, U1 MPU-6050, U2 DEV-16771, U3 LM7805_TO220, X1 ServoX, Y1 ServoY

Commit message: Add files via upload
Parts:
- added C1: 10uf, Capacitor_THT:CP_Radial_D5.0mm_P2.00mm, symbol Device:C
- added C2, C3, C4: 1uf, Capacitor_SMD:C_0603_1608Metric_Pad1.08x0.95mm_HandSolder, symbol Device:C
- added R10, R11: 1ohm, Resistor_THT:R_Axial_DIN0207_L6.3mm_D2.5mm_P10.16mm_Horizontal, symbol Device:R
- added R12: 1Mohm, Resistor_THT:R_Axial_DIN0207_L6.3mm_D2.5mm_P10.16mm_Horizontal, symbol Device:R
- added R13: 100kohm, Resistor_THT:R_Axial_DIN0207_L6.3mm_D2.5mm_P10.16mm_Horizontal, symbol Device:R
- added R9: 40ohm, Resistor_THT:R_Axial_DIN0207_L6.3mm_D2.5mm_P10.16mm_Horizontal, symbol Device:R
- 1ohm1, 1ohm2, 1ohm3, 1ohm4, 470ohm1, 470ohm2, 470ohm3, 470ohm4: footprint (none) -> Resistor_THT:R_Axial_DIN0207_L6.3mm_D2.5mm_P10.16mm_Horizontal
- AR1: renamed from ARM1; value Screw_Terminal_01x02 -> ARMING SWITCH; footprint (none) -> TerminalBlock:TerminalBlock_bornier-2_P5.08mm
- B1: footprint Package_LGA:Bosch_LGA-8_2x2.5mm_P0.65mm_ClockwisePinNumbering -> Connector_PinHeader_2.54mm:PinHeader_1x07_P2.54mm_Vertical
- BZ1: renamed from B1; footprint (none) -> Buzzer_Beeper:Buzzer_15x7.5RM7.6
- J1, J2, J3, J4: footprint (none) -> TerminalBlock:TerminalBlock_bornier-2_P5.08mm
- L1: footprint (none) -> LED_THT:LED_D5.0mm-4_RGB_Staggered_Pins
- P1: renamed from PWR1; value Screw_Terminal_01x02 -> PWR SWITCH; footprint (none) -> TerminalBlock:TerminalBlock_bornier-2_P5.08mm
- U1: footprint Sensor_Motion:InvenSense_QFN-24_4x4mm_P0.5mm -> Connector_PinHeader_2.54mm:PinHeader_1x08_P2.54mm_Vertical
- U2: footprint DEV-16771:MODULE_DEV-16771 -> Teensy 4.1:MODULE_DEV-16771
- X1, Y1: footprint (none) -> Connector_PinHeader_2.54mm:PinHeader_1x03_P2.54mm_Vertical
Connections:
- net +12V: now also J1.2 (Pin_2), J2.2 (Pin_2), J3.2 (Pin_2), J4.2 (Pin_2), P1.2 (Pin_2), R12.1; no longer U3.1 (VI)
- net +3V3: now also AR1.1 (Pin_1), C3.1, C4.1
- net GND: now also 470ohm1.1, 470ohm2.1, 470ohm3.1, BZ1.2 (+), Q1.3 (S), Q2.3 (S), Q3.3 (S), U2.GND1 (GND), U2.GND2 (GND), U2.GND3 (GND), U2.GND4 (GND), U2.GND5 (GND), U2.USB_GND1 (USB_GND), U2.USB_GND2 (USB_GND), C1.2, C2.2, C3.2, C4.2, R13.1
- net at L1.1 (A): now also U2.3.3V_1 (3.3V), U2.3.3V_2 (3.3V), U2.3.3V_3 (3.3V)
- net at L1.2 (RK): now also R9.2
- net at L1.3 (GK): now also R10.2
- net at L1.4 (BK): now also R11.2
- net at AR1.2 (Pin_2): now also U2.35 (TX8)
- net at U2.VIN, U3.3 (VO): now also C2.1
- net at U2.10 (CS1): now also F1.1 (~{CS})
- net at B1.3 (SDI), U1.24 (SDA), U2.18 (A4): now also F1.6 (CLK)
- net at U2.2 (OUT2): now also R11.1
- net at U2.3 (LRCLK2): now also F1.2 (DO(IO1))
- net at U2.34 (RX8): now also BZ1.1 (-)
- net at U2.4 (BCLK2): now also F1.5 (DI(IO0))
- net at U2.41 (A17): now also R12.2, R13.2
- net at U2.5 (IN2): now also U1.12 (INT)
- net at U2.6 (OUT1D): now also R9.1
- net at U2.9 (OUT1C): now also R10.1
- net at P1.1 (Pin_1): now also U3.1 (VI), C1.1
- no-connect marks 0 -> 51
Other:
- moved on the sheet: 1ohm1, 1ohm2, 1ohm3, 1ohm4, 470ohm1, 470ohm2, 470ohm3, 470ohm4, AR1, B1, BZ1, F1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
